File: ai03-pcb-guide-trial-1.kicad_pcb (KiCad board)
At the start: 2 copper layers, 94.5 x 57.2 mm, 34 parts, among them SW1 SW_Push, U1 ATmega32U4-AU, Y1 Crystal_GND24_Small

Commit message: Done designing (exporting next)
Routing:
- added copper zone on B.Cu, net GND
Other:
- board text added: "Hello World! by afs.7"
Changed lines of the file:
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@@
   (general
     (thickness 1.6)
-    (drawings 9)
+    (drawings 10)
     (tracks 276)
     (zones 0)
@@
       (rotate (xyz 0 0 0))
     )
+  )
+  (gr_text "Hello World! by afs.7" (at 150.8125 169.8625) (layer F.SilkS)
+    (effects (font (size 1 1) (thickness 0.15)))
   )
   (gr_line (start 132.55625 117.475) (end 137.31875 117.475) (layer Edge.Cuts) (width 0.05))
@@
   (segment (start 161.65475 152.90625) (end 161.43375 152.68525) (width 0.254) (layer B.Cu) (net 27))
   (segment (start 165.89375 152.90625) (end 161.65475 152.90625) (width 0.254) (layer B.Cu) (net 27))
+  (zone (net 1) (net_name GND) (layer B.Cu) (hatch edge 0.508)
+    (connect_pads (clearance 0.508))
+    (min_thickness 0.254)
+    (fill yes (arc_segments 32) (thermal_gap 0.508) (thermal_bridge_width 0.508))
+    (polygon
+      (pts
+        (xy 168.275 174.625) (xy 130.96875 174.625) (xy 130.96875 117.475) (xy 168.275 117.475)
+      )
+    )
+  )
 )
